File: BalanceFlex.kicad_pcb (KiCad board)
At the start: 2 copper layers, 306.2 x 100 mm, 9 parts, among them J1 Conn_01x10_Socket, J2 Conn_01x02_Socket, J3 Conn_01x01, J4 Conn_01x01, J5 Conn_01x01, J6 Conn_01x01, J7 Conn_01x01, J8 Conn_01x01, J9 Conn_01x01

Commit message: Cleaning up layout and adding in thermistors
Parts:
- added R1: R, Resistor_SMD:R_0402_1005Metric, F.Cu at (76.5, 98.1)
- added R2: R, Resistor_SMD:R_0402_1005Metric, F.Cu at (191.1, 97.6)
- added R3: R, Resistor_SMD:R_0402_1005Metric, F.Cu at (315.6, 98.0)
- added R4: R, Resistor_SMD:R_0402_1005Metric, F.Cu at (189.0, 186.0)
- moved J7 84.1 mm to (126.0, 178.0)
- moved J3 83.8 mm to (264.0, 178.0)
- moved J4 81.7 mm to (234.0, 102.0)
- moved J6 81.7 mm to (156.0, 102.0)
- moved J2 2.26 mm to (345.4, 114.9)
- moved J1 2.00 mm to (366.6, 127.0)
Connections:
- net Net-(J2-Pin_1) renamed GND
- J1 pad 2: unconnected-(J1-Pin_2-Pad2) -> Net-(J1-Pin_2)
- J1 pad 4: unconnected-(J1-Pin_4-Pad4) -> Net-(J1-Pin_4)
- J1 pad 7: unconnected-(J1-Pin_7-Pad7) -> Net-(J1-Pin_7)
- J1 pad 9: unconnected-(J1-Pin_9-Pad9) -> Net-(J1-Pin_9)
Routing:
- net Net-(J1-Pin_2): track 0.00 -> 322.5 mm, vias 0 -> 2
- net Net-(J1-Pin_9): track 0.00 -> 288.2 mm, vias 0 -> 2
- net Net-(J1-Pin_4): track 0.00 -> 205.1 mm, vias 0 -> 2
- net Net-(J1-Pin_10): track 162.8 -> 346.2 mm
- net Net-(J1-Pin_8): track 340.4 -> 164.7 mm
- net Net-(J1-Pin_1): track 236.6 -> 354.9 mm
- net Net-(J1-Pin_3): track 346.8 -> 249.5 mm
- net Net-(J1-Pin_7): track 0.00 -> 73.7 mm, vias 0 -> 2
- net Net-(J1-Pin_5): track 280.4 -> 286.0 mm
Other:
- board size 306.2 x 100 mm -> 308.2 x 100 mm

Commit message: had to add all files because I download zip instead of cloned
Parts:
- removed R1, R2, R3, R4: R, Resistor_SMD:R_0402_1005Metric
Connections:
- J1 pad 2: Net-(J1-Pin_2) -> Net-(J1-Pin_1)
- J1 pad 4: Net-(J1-Pin_4) -> Net-(J1-Pin_3)
- J1 pad 6: unconnected-(J1-Pin_6-Pad6) -> Net-(J1-Pin_5)
- J1 pad 8: Net-(J1-Pin_8) -> Net-(J1-Pin_7)
- J1 pad 9: Net-(J1-Pin_9) -> Net-(J1-Pin_10)
- J4 pad 1: Net-(J1-Pin_8) -> Net-(J1-Pin_7)
Routing:
- net Net-(J1-Pin_1): track 354.9 -> 17.4 mm
- net Net-(J1-Pin_2): track 322.5 -> 0.00 mm, vias 2 -> 0
- net Net-(J1-Pin_10): track 346.2 -> 24.5 mm
- net Net-(J1-Pin_9): track 288.2 -> 0.00 mm, vias 2 -> 0
- net Net-(J1-Pin_5): track 286.0 -> 20.2 mm
- net Net-(J1-Pin_3): track 249.5 -> 21.4 mm
- net Net-(J1-Pin_4): track 205.1 -> 0.00 mm, vias 2 -> 0
- net Net-(J1-Pin_8): track 164.7 -> 0.00 mm, vias 1 -> 0
- net Net-(J1-Pin_7): track 73.7 -> 21.4 mm, vias 2 -> 1
- added copper zone on In1.Cu, net Net-(J1-Pin_1)
- added copper zone on In1.Cu, net Net-(J1-Pin_10)
- added copper zone on In1.Cu, net Net-(J1-Pin_3)
- added copper zone on In2.Cu, net Net-(J1-Pin_5)
- added copper zone on In2.Cu, net Net-(J1-Pin_7)
Other:
- outline, holes or cut-outs redrawn
- copper layers 2 -> 4

Commit message: Tocuhing up
Routing:
- net Net-(J1-Pin_10): track 24.5 -> 1.41 mm, vias 1 -> 5
- added copper zone on F.Cu, net Net-(J1-Pin_10)
Other:
- outline, holes or cut-outs redrawn

Commit message: fillet + vias
Routing:
- net Net-(J1-Pin_3): track 21.4 -> 0.00 mm, vias 1 -> 4
- net Net-(J1-Pin_5): track 20.2 -> 0.00 mm, vias 1 -> 4
- net Net-(J1-Pin_7): track 21.4 -> 1.41 mm, vias 1 -> 5
- net Net-(J1-Pin_1): track 17.4 -> 0.00 mm, vias 1 -> 5
- added copper zone on F.Cu, net Net-(J1-Pin_1)
- added copper zone on F.Cu, net Net-(J1-Pin_3)
- added copper zone on F.Cu, net Net-(J1-Pin_5)
- added copper zone on F.Cu, net Net-(J1-Pin_7)
Other:
- outline, holes or cut-outs redrawn
